File: pcb/sigma-delta-dac-pcb/sigma-delta-dac-pcb.kicad_sch (KiCad schematic)
At the start: 17 parts, among them J1 Conn_02x03_Top_Bottom, J2 AudioJack3_SwitchTR, U1 Opamp_Dual

Commit message: OPAMP 출력단 저항 수정
Parts:
- R10, R5: value 50 -> 100
Changed lines of the file:
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@@
 			)
 		)
-		(property "Value" "50"
+		(property "Value" "100"
 			(at 142.24 129.54 90)
 			(show_name no)
@@
 			)
 		)
-		(property "Value" "50"
+		(property "Value" "100"
 			(at 142.24 82.55 90)
 			(show_name no)

Commit message: 회로도 수정: 50옴 롤백, OPAMP전원 캡 증가
Parts:
- C2: value 100nF -> 4.7uF
- R10, R5: value 100 -> 50
Changed lines of the file:
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@@
 			)
 		)
-		(property "Value" "100nF"
+		(property "Value" "4.7uF"
 			(at 85.09 49.5299 0)
 			(show_name no)
@@
 			)
 		)
-		(property "Value" "100"
+		(property "Value" "50"
 			(at 142.24 129.54 90)
 			(show_name no)
@@
 			)
 		)
-		(property "Value" "100"
+		(property "Value" "50"
 			(at 142.24 82.55 90)
 			(show_name no)

Commit message: v2 회로 - wip
Parts:
- removed C1: 100nF, Capacitor_SMD:C_0805_2012Metric_Pad1.18x1.45mm_HandSolder, symbol Device:C
- removed C2: 4.7uF, Capacitor_SMD:C_0805_2012Metric_Pad1.18x1.45mm_HandSolder, symbol Device:C
- removed C3, C7: 100uF, Capacitor_SMD:CP_Elec_6.3x5.3, symbol Device:C_Polarized
- removed C4, C8: 22nF, Capacitor_SMD:C_0805_2012Metric_Pad1.18x1.45mm_HandSolder, symbol Device:C
- removed C5, C9: 2.2nF, Capacitor_SMD:C_0805_2012Metric_Pad1.18x1.45mm_HandSolder, symbol Device:C
- removed J1: Conn_02x03_Top_Bottom, Connector_PinSocket_2.54mm:PinSocket_2x03_P2.54mm_Vertical, symbol Connector_Generic:Conn_02x03_Top_Bottom
- removed J2: AudioJack3_SwitchTR, Connector_Audio:Jack_3.5mm_CUI_SJ1-3525N_Horizontal, symbol Connector_Audio:AudioJack3_SwitchTR
- removed R10, R5: 50, Resistor_SMD:R_0805_2012Metric_Pad1.20x1.40mm_HandSolder, symbol Device:R_US
- removed R3, R8: 220, Resistor_SMD:R_0805_2012Metric_Pad1.20x1.40mm_HandSolder, symbol Device:R_US
- removed R4, R9: 2.2k, Resistor_SMD:R_0805_2012Metric_Pad1.20x1.40mm_HandSolder, symbol Device:R_US
- removed U1: Opamp_Dual, Package_SO:SOIC-8_3.9x4.9mm_P1.27mm, symbol Device:Opamp_Dual
Other:
- added sheet Conn (conn.kicad_sch)
- added sheet Filter (filter.kicad_sch)
- added sheet Power (power.kicad_sch)
- added sheet Sim (sim.kicad_sch)
