File: pcb/sigma-delta-dac-pcb/conn.kicad_sch (KiCad schematic)
At the start: 6 parts, among them J1 Conn_02x03_Top_Bottom, J2 AudioJack3_SwitchTR

Commit message: V2 보드 완성
Other:
- moved on the sheet: R2
Changed lines of the file:
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@@
 	(wire
 		(pts
-			(xy 39.37 66.04) (xy 43.18 66.04)
+			(xy 39.37 76.2) (xy 43.18 76.2)
 		)
 		(stroke
@@
 	(wire
 		(pts
-			(xy 50.8 57.15) (xy 55.88 57.15)
+			(xy 50.8 57.15) (xy 69.85 57.15)
 		)
 		(stroke
@@
 	(wire
 		(pts
-			(xy 50.8 66.04) (xy 55.88 66.04)
+			(xy 50.8 76.2) (xy 69.85 76.2)
 		)
 		(stroke
@@
 	(global_label "SDM_L"
 		(shape input)
-		(at 55.88 57.15 0)
+		(at 69.85 57.15 0)
 		(fields_autoplaced yes)
 		(effects
@@
 		)
 		(property "Intersheetrefs" "${INTERSHEET_REFS}"
-			(at 64.7918 57.15 0)
+			(at 78.7618 57.15 0)
 			(hide yes)
 			(show_name no)
@@
 	(global_label "SDM_R_IN"
 		(shape input)
-		(at 39.37 66.04 180)
+		(at 39.37 76.2 180)
 		(fields_autoplaced yes)
 		(effects
@@
 		)
 		(property "Intersheetrefs" "${INTERSHEET_REFS}"
-			(at 27.3134 66.04 0)
+			(at 27.3134 76.2 0)
 			(hide yes)
 			(show_name no)
@@
 	(global_label "SDM_R"
 		(shape input)
-		(at 55.88 66.04 0)
+		(at 69.85 76.2 0)
 		(fields_autoplaced yes)
 		(effects
@@
 		)
 		(property "Intersheetrefs" "${INTERSHEET_REFS}"
-			(at 65.0337 66.04 0)
+			(at 79.0037 76.2 0)
 			(hide yes)
 			(show_name no)
@@
 		(unit 1)
 		(body_style 1)
-		(exclude_from_sim no)
+		(exclude_from_sim yes)
 		(in_bom no)
 		(on_board yes)
@@
 		(unit 1)
 		(body_style 1)
-		(exclude_from_sim no)
+		(exclude_from_sim yes)
 		(in_bom no)
 		(on_board yes)
@@
 	(symbol
 		(lib_id "Device:R_US")
-		(at 46.99 66.04 90)
+		(at 46.99 76.2 90)
 		(unit 1)
 		(body_style 1)
@@
 		(fields_autoplaced yes)
 		(property "Reference" "R2"
-			(at 46.99 59.69 90)
+			(at 46.99 69.85 90)
 			(show_name no)
 			(do_not_autoplace no)
@@
 		)
 		(property "Value" "0"
-			(at 46.99 62.23 90)
+			(at 46.99 72.39 90)
 			(show_name no)
 			(do_not_autoplace no)
@@
 		)
 		(property "Footprint" "Resistor_SMD:R_0805_2012Metric_Pad1.20x1.40mm_HandSolder"
-			(at 47.244 65.024 90)
+			(at 47.244 75.184 90)
 			(hide yes)
 			(show_name no)
@@
 		)
 		(property "Datasheet" ""
-			(at 46.99 66.04 0)
+			(at 46.99 76.2 0)
 			(hide yes)
 			(show_name no)
@@
 		)
 		(property "Description" "Resistor, US symbol"
-			(at 46.99 66.04 0)
-			(hide yes)
-			(show_name no)
+			(at 46.99 76.2 0)
+			(hide yes)
+			(show_name no)
