File: pcb/sigma-delta-dac-pcb/conn.kicad_sch (KiCad schematic)
At the start: 6 parts, among them J1 Conn_02x03_Top_Bottom, J2 AudioJack3_SwitchTR

Commit message: V3 보드 WIP
Parts:
- R1, R2: value 0 -> 330; footprint Resistor_SMD:R_0805_2012Metric_Pad1.20x1.40mm_HandSolder -> Resistor_SMD:R_0603_1608Metric
- renumbered J2 to J1, J1 to J2
Other:
- moved on the sheet: J1
Changed lines of the file:
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@@
 	(paper "A4")
 	(junction
-		(at 77.47 106.68)
+		(at 154.94 38.1)
 		(diameter 0)
 		(color 0 0 0 0)
 	)
 	(junction
-		(at 77.47 101.6)
+		(at 154.94 33.02)
 		(diameter 0)
 		(color 0 0 0 0)
@@
 	(wire
 		(pts
-			(xy 76.2 99.06) (xy 93.98 99.06)
+			(xy 153.67 30.48) (xy 171.45 30.48)
 		)
 		(stroke
@@
 	(wire
 		(pts
-			(xy 76.2 106.68) (xy 77.47 106.68)
-		)
-		(stroke
-			(width 0)
-			(type default)
-		)
-	)
-	(wire
-		(pts
-			(xy 77.47 101.6) (xy 93.98 101.6)
-		)
-		(stroke
-			(width 0)
-			(type default)
-		)
-	)
-	(wire
-		(pts
-			(xy 76.2 109.22) (xy 77.47 109.22)
-		)
-		(stroke
-			(width 0)
-			(type default)
-		)
-	)
-	(wire
-		(pts
-			(xy 76.2 104.14) (xy 77.47 104.14)
-		)
-		(stroke
-			(width 0)
-			(type default)
-		)
-	)
-	(wire
-		(pts
-			(xy 77.47 109.22) (xy 77.47 106.68)
+			(xy 153.67 38.1) (xy 154.94 38.1)
+		)
+		(stroke
+			(width 0)
+			(type default)
+		)
+	)
+	(wire
+		(pts
+			(xy 154.94 33.02) (xy 171.45 33.02)
+		)
+		(stroke
+			(width 0)
+			(type default)
+		)
+	)
+	(wire
+		(pts
+			(xy 153.67 40.64) (xy 154.94 40.64)
+		)
+		(stroke
+			(width 0)
+			(type default)
+		)
+	)
+	(wire
+		(pts
+			(xy 153.67 35.56) (xy 154.94 35.56)
+		)
+		(stroke
+			(width 0)
+			(type default)
+		)
+	)
+	(wire
+		(pts
+			(xy 154.94 40.64) (xy 154.94 38.1)
 		)
 		(stroke
@@
 	(wire
 		(pts
-			(xy 77.47 106.68) (xy 93.98 106.68)
+			(xy 154.94 38.1) (xy 171.45 38.1)
 		)
 		(stroke
@@
 	(wire
 		(pts
-			(xy 76.2 101.6) (xy 77.47 101.6)
-		)
-		(stroke
-			(width 0)
-			(type default)
-		)
-	)
-	(wire
-		(pts
-			(xy 77.47 104.14) (xy 77.47 101.6)
+			(xy 153.67 33.02) (xy 154.94 33.02)
+		)
+		(stroke
+			(width 0)
+			(type default)
+		)
+	)
+	(wire
+		(pts
+			(xy 154.94 35.56) (xy 154.94 33.02)
 		)
 		(stroke
@@
 	(global_label "A_OUT_R"
 		(shape input)
-		(at 93.98 101.6 0)
+		(at 171.45 33.02 0)
 		(fields_autoplaced yes)
 		(effects
@@
 		)
 		(property "Intersheetrefs" "${INTERSHEET_REFS}"
-			(at 104.8876 101.6 0)
+			(at 182.3576 33.02 0)
 			(hide yes)
 			(show_name no)
@@
 	(global_label "A_OUT_L"
 		(shape input)
-		(at 93.98 106.68 0)
+		(at 171.45 38.1 0)
 		(fields_autoplaced yes)
 		(effects
@@
 		)
 		(property "Intersheetrefs" "${INTERSHEET_REFS}"
-			(at 104.6457 106.68 0)
+			(at 182.1157 38.1 0)
 			(hide yes)
 			(show_name no)
@@
 		(dnp no)
 		(fields_autoplaced yes)
-		(property "Reference" "#PWR02"
+		(property "Reference" "#PWR03"
 			(at 27.94 36.83 0)
 			(hide yes)
@@
 			(project "sigma-delta-dac-pcb"
 				(path "/a35bdaff-6288-40da-b7db-a5834010c771/65e66474-56ea-44cd-957a-a0d1d78aa642"
-					(reference "#PWR02")
+					(reference "#PWR03")
 					(unit 1)
 				)
@@
 		(dnp no)
 		(fields_autoplaced yes)
-		(property "Reference" "#PWR01"
+		(property "Reference" "#PWR02"
 			(at 67.31 31.75 0)
 			(hide yes)
@@
 			(project "sigma-delta-dac-pcb"
 				(path "/a35bdaff-6288-40da-b7db-a5834010c771/65e66474-56ea-44cd-957a-a0d1d78aa642"
-					(reference "#PWR01")
+					(reference "#PWR02")
 					(unit 1)
 				)
@@
 	(symbol
 		(lib_id "power:GND")
-		(at 93.98 99.06 90)
+		(at 171.45 30.48 90)
 		(unit 1)
 		(body_style 1)
@@
 		(dnp no)
 		(fields_autoplaced yes)
-		(property "Reference" "#PWR03"
-			(at 100.33 99.06 0)
+		(property "Reference" "#PWR01"
+			(at 177.8 30.48 0)
 			(hide yes)
 			(show_name no)
@@
 		)
 		(property "Value" "GND"
-			(at 97.79 99.0599 90)
+			(at 175.26 30.4799 90)
 			(show_name no)
 			(do_not_autoplace no)
@@
 		)
 		(property "Footprint" ""
-			(at 93.98 99.06 0)
+			(at 171.45 30.48 0)
 			(hide yes)
 			(show_name no)
@@
 		)
 		(property "Datasheet" ""
-			(at 93.98 99.06 0)
+			(at 171.45 30.48 0)
 			(hide yes)
 			(show_name no)
@@
 		)
 		(property "Description" "Power symbol creates a global label with name \"GND\" , ground"
-			(at 93.98 99.06 0)
+			(at 171.45 30.48 0)
 			(hide yes)
 			(show_name no)
@@
 			(project "sigma-delta-dac-pcb"
 				(path "/a35bdaff-6288-40da-b7db-a5834010c771/65e66474-56ea-44cd-957a-a0d1d78aa642"
-					(reference "#PWR03")
+					(reference "#PWR01")
 					(unit 1)
 				)
@@
 		(unit 1)
 		(body_style 1)
-		(exclude_from_sim yes)
+		(exclude_from_sim no)
 		(in_bom yes)
 		(on_board yes)
@@
 		(dnp no)
 		(fields_autoplaced yes)
-		(property "Reference" "J1"
+		(property "Reference" "J2"
 			(at 46.99 25.4 0)
 			(show_name no)
@@
 			(project "sigma-delta-dac-pcb"
 				(path "/a35bdaff-6288-40da-b7db-a5834010c771/65e66474-56ea-44cd-957a-a0d1d78aa642"
-					(reference "J1")
+					(reference "J2")
 					(unit 1)
 				)
@@
 		(in_pos_files yes)
 		(dnp no)
-		(fields_autoplaced yes)
 		(property "Reference" "R2"
 			(at 46.99 69.85 90)
@@
 			)
 		)
-		(property "Value" "0"
+		(property "Value" "330"
 			(at 46.99 72.39 90)
 			(show_name no)
@@
 			)
 		)
-		(property "Footprint" "Resistor_SMD:R_0805_2012Metric_Pad1.20x1.40mm_HandSolder"
+		(property "Footprint" "Resistor_SMD:R_0603_1608Metric"
 			(at 47.244 75.184 90)
 			(hide yes)
@@
 			)
 		)
-		(property "Description" "Resistor, US symbol"
-			(at 46.99 76.2 0)
-			(hide yes)
+		(property "Description" "1608"
+			(at 46.99 74.422 90)
 			(show_name no)
 			(do_not_autoplace no)
@@
 		(in_pos_files yes)
 		(dnp no)
-		(fields_autoplaced yes)
 		(property "Reference" "R1"
 			(at 46.99 50.8 90)
@@
 			)
 		)
-		(property "Value" "0"
+		(property "Value" "330"
 			(at 46.99 53.34 90)
 			(show_name no)
@@
 			)
 		)
-		(property "Footprint" "Resistor_SMD:R_0805_2012Metric_Pad1.20x1.40mm_HandSolder"
+		(property "Footprint" "Resistor_SMD:R_0603_1608Metric"
 			(at 47.244 56.134 90)
 			(hide yes)
@@
 			)
 		)
-		(property "Description" "Resistor, US symbol"
-			(at 46.99 57.15 0)
-			(hide yes)
+		(property "Description" "1608"
+			(at 46.99 55.372 90)
 			(show_name no)
 			(do_not_autoplace no)
@@
 	(symbol
 		(lib_id "Connector_Audio:AudioJack3_SwitchTR")
-		(at 71.12 101.6 0)
+		(at 148.59 33.02 0)
 		(unit 1)
 		(body_style 1)
-		(exclude_from_sim yes)
+		(exclude_from_sim no)
 		(in_bom yes)
 		(on_board yes)
@@
 		(dnp no)
 		(fields_autoplaced yes)
-		(property "Reference" "J2"
-			(at 69.215 92.71 0)
+		(property "Reference" "J1"
+			(at 146.685 24.13 0)
 			(show_name no)
 			(do_not_autoplace no)
@@
 		)
 		(property "Value" "AudioJack3_SwitchTR"
-			(at 69.215 95.25 0)
+			(at 146.685 26.67 0)
 			(show_name no)
 			(do_not_autoplace no)
@@
 		)
 		(property "Footprint" "Connector_Audio:Jack_3.5mm_CUI_SJ1-3525N_Horizontal"
-			(at 71.12 101.6 0)
+			(at 148.59 33.02 0)
 			(hide yes)
 			(show_name no)
@@
 		)
 		(property "Datasheet" ""
-			(at 71.12 101.6 0)
+			(at 148.59 33.02 0)
 			(hide yes)
 			(show_name no)
@@
 		)
 		(property "Description" "Audio Jack, 3 Poles (Stereo / TRS), Switched TR Poles (Normalling)"
-			(at 71.12 101.6 0)
+			(at 148.59 33.02 0)
 			(hide yes)
 			(show_name no)
@@
 			(project "sigma-delta-dac-pcb"
 				(path "/a35bdaff-6288-40da-b7db-a5834010c771/65e66474-56ea-44cd-957a-a0d1d78aa642"
-					(reference "J2")
+					(reference "J1")
 					(unit 1)
 				)

Commit message: BOM 정리
Changed lines of the file:
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@@
 			)
 		)
-		(property "Description" "1608"
+		(property "Description" "1608 1%"
 			(at 46.99 74.422 90)
 			(show_name no)
@@
 			)
 		)
-		(property "Description" "1608"
+		(property "Description" "1608 1%"
 			(at 46.99 55.372 90)
 			(show_name no)
