File: pcb/sigma-delta-dac-pcb/filter.kicad_sch (KiCad schematic)
At the start: 15 parts, among them U2 TLV9062

Commit message: V3 보드 WIP
Parts:
- removed C10, C5: 100uF, Capacitor_SMD:CP_Elec_6.3x5.3, symbol Device:C_Polarized
- removed C11, C8: 22nF, Capacitor_SMD:C_0805_2012Metric_Pad1.18x1.45mm_HandSolder, symbol Device:C
- removed C6, C7: 100nF, Capacitor_SMD:C_0805_2012Metric_Pad1.18x1.45mm_HandSolder, symbol Device:C
- removed C9: 2.2nF, Capacitor_SMD:C_0805_2012Metric_Pad1.18x1.45mm_HandSolder, symbol Device:C
- removed R10: 50, Resistor_SMD:R_0805_2012Metric_Pad1.20x1.40mm_HandSolder, symbol Device:R_US
- removed R5, R8: 220, Resistor_SMD:R_0805_2012Metric_Pad1.20x1.40mm_HandSolder, symbol Device:R_US
- removed R6, R9: 2.2k, Resistor_SMD:R_0805_2012Metric_Pad1.20x1.40mm_HandSolder, symbol Device:R_US
- removed U2: TLV9062, Package_SO:SOIC-8_3.9x4.9mm_P1.27mm, symbol Amplifier_Operational:TLV9062
- added C13, C15: 1 nF, Capacitor_SMD:C_0603_1608Metric, symbol Device:C
- added C14: 2.2nF, Capacitor_SMD:C_0603_1608Metric, symbol Device:C
- added C16, C17: 100nF, Capacitor_SMD:C_0603_1608Metric, symbol Device:C
- added R11, R14: 2.61k, Resistor_SMD:R_0603_1608Metric, symbol Device:R_US
- added R12, R15: 4.87k, Resistor_SMD:R_0603_1608Metric, symbol Device:R_US
- added R16: 0, Resistor_SMD:R_0805_2012Metric, symbol Device:R_US
- added U4: OPA1688IDR, Package_SO:SOIC-8_3.9x4.9mm_P1.27mm, symbol OPA1688IDR:OPA1688IDR
- C12: footprint Capacitor_SMD:C_0805_2012Metric_Pad1.18x1.45mm_HandSolder -> Capacitor_SMD:C_0603_1608Metric
- R13: renamed from R7; value 50 -> 0; footprint Resistor_SMD:R_0805_2012Metric_Pad1.20x1.40mm_HandSolder -> Resistor_SMD:R_0805_2012Metric
Connections:
- net A_OUT_L: now also R13.2
- net A_OUT_R: now also R16.2
- net GND: now also C13.1, C15.1, C16.2, C17.1; no longer C12.2
- net at C12.1: now also R11.2, R12.1
- net at R13.1: now also C12.2, U4.1, U4.2 (-)
- new net: C13.2, R12.2, U4.3 (+)
- new net: C14.1, R14.2, R15.1
- new net: C14.2, R16.1, U4.6 (-), U4.7
- new net: C15.2, R15.2, U4.5 (+)
- new net +3V3: C16.1, U4.8 (V+)
- new net -3V3: C17.2, U4.4 (V-)
- new net BUFFER_L: R11.1
- new net BUFFER_R: R14.1
Other:
- moved on the sheet: R13

Commit message: 캐패시터 사이즈 변경
Parts:
- C16, C17: footprint Capacitor_SMD:C_0603_1608Metric -> Capacitor_SMD:C_0402_1005Metric

Commit message: 아트웍 wip
Connections:
- net at C12.1, R11.2: now also R12.2; no longer R12.1
- net at C13.2, U4.3 (+): now also R12.1; no longer R12.2
Other:
- moved on the sheet: R12
Changed lines of the file:
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@@
 	(symbol
 		(lib_id "Device:R_US")
-		(at 123.19 34.29 90)
+		(at 123.19 34.29 270)
+		(mirror x)
 		(unit 1)
 		(body_style 1)
@@
 		(dnp no)
 		(property "Reference" "R12"
-			(at 121.9199 31.75 0)
+			(at 124.4601 31.75 0)
 			(show_name no)
 			(do_not_autoplace no)
@@
 		)
 		(property "Value" "4.87k"
-			(at 124.4599 31.75 0)
+			(at 121.9201 31.75 0)
 			(show_name no)
 			(do_not_autoplace no)
@@
 		)
 		(property "Footprint" "Resistor_SMD:R_0603_1608Metric"
-			(at 123.444 33.274 90)
+			(at 122.936 33.274 90)
 			(hide yes)
 			(show_name no)
@@
 		)
 		(property "Description" "1608 1%"
-			(at 126.492 27.432 0)
+			(at 119.888 27.432 0)
 			(show_name no)
 			(do_not_autoplace no)

Commit message: 레이아웃 최적화, opamp 캐패시터 추가
Parts:
- added C16, C18: 100nF, Capacitor_SMD:C_0402_1005Metric, symbol Device:C
- renumbered C16 to C17, C17 to C19
Connections:
- net +3V3: now also C16.1
- net -3V3: now also C18.2
- net GND: now also C16.2, C18.1
