File: pcb/sigma-delta-dac-pcb/power.kicad_sch (KiCad schematic)
At the start: 4 parts

Commit message: V2 보드 완성
Parts:
- removed R3: 0, Resistor_SMD:R_0805_2012Metric_Pad1.20x1.40mm_HandSolder, symbol Device:R_US
- added C2, C4: 100uF, Capacitor_Tantalum_SMD:CP_EIA-3528-15_AVX-H_HandSolder, symbol Device:C_Polarized
- added FB1: (no value), Inductor_SMD:L_0805_2012Metric_Pad1.05x1.20mm_HandSolder, symbol Device:FerriteBead
- renumbered C2 to C3
Connections:
- net 5V_IN: now also C1.1, C2.1, FB1.1
- net GND: now also C2.2, C4.2
- net at C3.1, R4.2: now also C4.1, FB1.2; no longer C1.1
Other:
- moved on the sheet: R4
