File: pcb/sigma-delta-dac-pcb/power.kicad_sch (KiCad schematic)
At the start: 11 parts, among them U1 LM27762

Commit message: 캐패시터 사이즈 변경
Parts:
- C1, C3: footprint Capacitor_SMD:C_0805_2012Metric -> Capacitor_SMD:C_0603_1608Metric
- C2, C4, C5: footprint Capacitor_SMD:C_0603_1608Metric -> Capacitor_SMD:C_0402_1005Metric
Changed lines of the file:
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@@
 			)
 		)
-		(property "Footprint" "Capacitor_SMD:C_0603_1608Metric"
+		(property "Footprint" "Capacitor_SMD:C_0402_1005Metric"
 			(at 88.5952 95.25 0)
 			(hide yes)
@@
 			)
 		)
-		(property "Description" "25V X7R 1608"
+		(property "Description" "16V X5R 1005"
 			(at 96.52 95.758 0)
 			(show_name no)
@@
 			)
 		)
-		(property "Footprint" "Capacitor_SMD:C_0805_2012Metric"
+		(property "Footprint" "Capacitor_SMD:C_0603_1608Metric"
 			(at 60.6552 46.99 0)
 			(hide yes)
@@
 			)
 		)
-		(property "Description" "2012 50V X5R"
+		(property "Description" "1608 10V X7R"
 			(at 66.802 46.482 0)
 			(show_name no)
@@
 			)
 		)
-		(property "Footprint" "Capacitor_SMD:C_0603_1608Metric"
+		(property "Footprint" "Capacitor_SMD:C_0402_1005Metric"
 			(at 33.9852 93.98 0)
 			(hide yes)
@@
 			)
 		)
-		(property "Description" "16V 1608 X7R"
+		(property "Description" "16V 1005 X5R"
 			(at 41.402 93.218 0)
 			(show_name no)
@@
 			)
 		)
-		(property "Footprint" "Capacitor_SMD:C_0603_1608Metric"
+		(property "Footprint" "Capacitor_SMD:C_0402_1005Metric"
 			(at 111.4552 95.25 0)
 			(hide yes)
@@
 			)
 		)
-		(property "Description" "25V X7R 1608"
+		(property "Description" "16V X5R 1005"
 			(at 120.142 95.504 0)
 			(show_name no)
@@
 			)
 		)
-		(property "Footprint" "Capacitor_SMD:C_0805_2012Metric"
+		(property "Footprint" "Capacitor_SMD:C_0603_1608Metric"
 			(at 55.5752 95.25 0)
 			(hide yes)
@@
 			)
 		)
-		(property "Description" "2012 50V X5R"
+		(property "Description" "1608 10V X7R"
 			(at 61.722 94.742 0)
 			(show_name no)

Commit message: 레이아웃 최적화, opamp 캐패시터 추가
Parts:
- added TP1, TP2, TP3, TP4: TestPoint, TestPoint:TestPoint_Pad_1.0x1.0mm, symbol Connector:TestPoint
Connections:
- net +3V3: now also TP1.1
- net -3V3: now also TP3.1
- net GND: now also TP2.1, TP4.1

Commit message: BOM 정리
Parts:
- TP1, TP2, TP3, TP4: now left out of the parts list
Changed lines of the file:
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@@
 		(body_style 1)
 		(exclude_from_sim no)
-		(in_bom yes)
+		(in_bom no)
 		(on_board yes)
 		(in_pos_files yes)
@@
 		(body_style 1)
 		(exclude_from_sim no)
-		(in_bom yes)
+		(in_bom no)
 		(on_board yes)
 		(in_pos_files yes)
@@
 		(body_style 1)
 		(exclude_from_sim no)
-		(in_bom yes)
+		(in_bom no)
 		(on_board yes)
 		(in_pos_files yes)
@@
 		(body_style 1)
 		(exclude_from_sim no)
-		(in_bom yes)
-		(on_board yes)
-		(in_pos_files yes)
+		(in_bom no)
+		(on_board yes)
+		(in_pos_files yes)
