File: pcb/sigma-delta-dac-pcb/sigma-delta-dac-pcb.kicad_pcb (KiCad board)
At the start: 2 copper layers, 60 x 32.5 mm, 19 parts, among them J1 Conn_02x03_Top_Bottom, J2 AudioJack3_SwitchTR, U1 Opamp_Dual

Commit message: 시뮬레이션 수정
Parts:
- C2: value 100nF -> 4.7uF
Connections:
- net /+3V3 renamed +3V3
- net /A_OUT_L renamed A_OUT_L
- net /A_OUT_R renamed A_OUT_R
- net /SDM_L renamed SDM_L
- net /SDM_R renamed SDM_R

Commit message: v2 회로 - wip
Parts:
- removed REF** (x2): MountingHole_3mm, MountingHole:MountingHole_3mm
- removed U1: Opamp_Dual, Package_SO:SOIC-8_3.9x4.9mm_P1.27mm
- added C10: 2.2nF, Capacitor_SMD:C_0805_2012Metric_Pad1.18x1.45mm_HandSolder, F.Cu at (112.0, 101.3)
- added C6: 22nF, Capacitor_SMD:C_0805_2012Metric_Pad1.18x1.45mm_HandSolder, F.Cu at (107.8, 112.5)
- added H1: MountingHole, MountingHole:MountingHole_3.2mm_M3, F.Cu at (144.5, 90.8)
- added H2: MountingHole, MountingHole:MountingHole_3.2mm_M3, F.Cu at (144.5, 114.2)
- added R1: 0, Resistor_SMD:R_0805_2012Metric_Pad1.20x1.40mm_HandSolder, F.Cu at (102.5, 109.2)
- added R2: 0, Resistor_SMD:R_0805_2012Metric_Pad1.20x1.40mm_HandSolder, F.Cu at (102.5, 104.8)
- added R6: 2.2k, Resistor_SMD:R_0805_2012Metric_Pad1.20x1.40mm_HandSolder, F.Cu at (111.0, 109.2)
- added R7: 50, Resistor_SMD:R_0805_2012Metric_Pad1.20x1.40mm_HandSolder, F.Cu at (116.5, 98.8)
- added U2: TLV9062, Package_SO:SOIC-8_3.9x4.9mm_P1.27mm, F.Cu at (118.2, 104.2)
- C2: value 4.7uF -> 100nF
- C4: value 22nF -> 100nF
- C5: value 2.2nF -> 100nF
- C7: value 100uF -> 2.2nF; footprint Capacitor_SMD:CP_Elec_6.3x5.3 -> Capacitor_SMD:C_0805_2012Metric_Pad1.18x1.45mm_HandSolder
- C8: value 22nF -> 100uF; footprint Capacitor_SMD:C_0805_2012Metric_Pad1.18x1.45mm_HandSolder -> Capacitor_SMD:CP_Elec_6.3x5.3
- C9: value 2.2nF -> 22nF
- R3: value 220 -> 0
- R4: value 2.2k -> 0
- R5: value 50 -> 220
- moved C8 29.8 mm to (132.9, 113.2), turned to 0 degrees
- moved C1 29.6 mm to (101.5, 90.0), turned to 90 degrees
- moved C2 25.8 mm to (104.5, 90.0), turned to 90 degrees
- moved C7 20.0 mm to (112.0, 112.5), turned to -90 degrees
- moved C4 18.9 mm to (124.8, 101.6), turned to 0 degrees
- moved R5 16.9 mm to (106.8, 109.2)
- moved R4 16.2 mm to (113.5, 90.0), turned to 180 degrees
- moved R3 13.2 mm to (93.5, 96.0), turned to -90 degrees
- moved C5 12.3 mm to (124.8, 99.0), turned to 0 degrees
- moved C9 7.95 mm to (107.8, 101.2)
- moved R10 5.67 mm to (124.8, 108.8), turned to -90 degrees
- moved R8 4.65 mm to (106.8, 104.8)
- moved R9 4.25 mm to (111.0, 104.8)
- moved J1 1.10 mm to (93.5, 100.5)
- moved C3 1.06 mm to (133.2, 91.2)
Connections:
- net +3V3 renamed 3.3V_IN
- C1 pad 1: +5V -> Net-(C1-Pad1)
- C2 pad 1: +5V -> Net-(C1-Pad1)
- C4 pad 1: Net-(C4-Pad1) -> +5V
- C5 pad 1: Net-(U1A-+) -> +5V
- C7 pad 1: Net-(C7-Pad1) -> Net-(U2A-+)
- C7 pad 2: A_OUT_R -> GND
- C8 pad 2: GND -> A_OUT_R
- C9 pad 1: Net-(U1B-+) -> Net-(C9-Pad1)
- J1 pad 1: +5V -> 5V_IN
- J1 pad 5: SDM_L -> SDM_L_IN
- J1 pad 6: SDM_R -> SDM_R_IN
- J2 pad RN: unconnected-(J2-PadRN) -> A_OUT_R
- J2 pad TN: unconnected-(J2-PadTN) -> A_OUT_L
- R10 pad 2: Net-(C7-Pad1) -> Net-(C8-Pad1)
- R3 pad 1: SDM_L -> Net-(C1-Pad1)
- R3 pad 2: Net-(C4-Pad1) -> 5V_IN
- R4 pad 1: Net-(C4-Pad1) -> +5V
- R4 pad 2: Net-(U1A-+) -> Net-(C1-Pad1)
- R5 pad 1: Net-(U1A--) -> SDM_L
- R5 pad 2: Net-(C3-Pad1) -> Net-(C6-Pad1)
- R8 pad 2: Net-(C8-Pad1) -> Net-(C9-Pad1)
- R9 pad 1: Net-(C8-Pad1) -> Net-(C9-Pad1)
- R9 pad 2: Net-(U1B-+) -> Net-(U2B-+)
Routing:
- net Net-(C1-Pad1): track 0.00 -> 21.9 mm
- net Net-(U1B-+): track 17.4 -> 0.00 mm, vias 2 -> 0
- net Net-(U2B-+): track 0.00 -> 15.5 mm, vias 0 -> 2
- net +5V: track 34.9 -> 20.8 mm, vias 1 -> 0
- net GND: track 0.00 -> 12.9 mm, vias 33 -> 42
- net Net-(C7-Pad1): track 9.74 -> 0.00 mm
- net SDM_L_IN: track 0.00 -> 9.58 mm
- net SDM_L: track 11.4 -> 2.25 mm
- net Net-(U1A-+): track 8.80 -> 0.00 mm
- net Net-(U2A-+): track 0.00 -> 8.53 mm
- net Net-(C4-Pad1): track 7.19 -> 0.00 mm
- net SDM_R_IN: track 0.00 -> 6.12 mm
- net SDM_R: track 7.98 -> 2.25 mm
- net Net-(C3-Pad1): track 13.6 -> 18.5 mm
- net Net-(C9-Pad1): track 0.00 -> 4.71 mm
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- removed copper zone on F.Cu, net +5V
Other:
- board text added: "Sigma-Delta-V2"
- board text removed: "3.3V"
- board text removed: "5V"
- board text removed: "GND"
- board text removed: "IN_L"
- board text removed: "IN_R"
- board text removed: "Sigma-Delta-V1"

Commit message: Via 추가
Routing:
- net GND: vias 42 -> 43
Changed lines of the file:
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@@
+	)
+	(via
+		(at 120.5 98)
+		(size 0.5)
+		(drill 0.3)
+		(layers "F.Cu" "B.Cu")
+		(net "GND")
 	)
 	(via
@@
 		(layer "B.Cu")
 		(net "Net-(C3-Pad1)")
+	)
+	(segment
+		(start 100.5375 92)
+		(end 101.5 91.0375)
+		(width 0.4)
+		(layer "F.Cu")
+		(net "Net-(C1-Pad1)")
+	)
+	(segment
+		(start 93.5 93.6)
+		(end 95.1 92)
+		(width 0.4)
+		(layer "F.Cu")
+		(net "Net-(C1-Pad1)")
+	)
+	(segment
+		(start 107.5 90)
+		(end 112.5 90)
+		(width 0.4)
+		(layer "F.Cu")
+		(net "Net-(C1-Pad1)")
+	)
+	(segment
+		(start 93.5 95)
+		(end 93.5 93.6)
+		(width 0.4)
+		(layer "F.Cu")
+		(net "Net-(C1-Pad1)")
+	)
+	(segment
+		(start 95.1 92)
+		(end 100.5375 92)
+		(width 0.4)
+		(layer "F.Cu")
+		(net "Net-(C1-Pad1)")
+	)
+	(segment
+		(start 106.4625 91.0375)
+		(end 107.5 90)
+		(width 0.4)
+		(layer "F.Cu")
+		(net "Net-(C1-Pad1)")
+	)
+	(segment
+		(start 104.5 91.0375)
+		(end 106.4625 91.0375)
+		(width 0.4)
+		(layer "F.Cu")
+		(net "Net-(C1-Pad1)")
+	)
+	(segment
+		(start 101.5 91.0375)
+		(end 104.5 91.0375)
+		(width 0.4)
+		(layer "F.Cu")
+		(net "Net-(C1-Pad1)")
 	)
 	(segment
@@
 		(net "A_OUT_L")
 	)
-	(segment
-		(start 100.5375 92)
-		(end 101.5 91.0375)
-		(width 0.4)
-		(layer "F.Cu")
-		(net "Net-(C1-Pad1)")
-	)
-	(segment
-		(start 93.5 93.6)
-		(end 95.1 92)
-		(width 0.4)
-		(layer "F.Cu")
-		(net "Net-(C1-Pad1)")
-	)
-	(segment
-		(start 107.5 90)
-		(end 112.5 90)
-		(width 0.4)
-		(layer "F.Cu")
-		(net "Net-(C1-Pad1)")
-	)
-	(segment
-		(start 93.5 95)
-		(end 93.5 93.6)
-		(width 0.4)
-		(layer "F.Cu")
-		(net "Net-(C1-Pad1)")
-	)
-	(segment
-		(start 95.1 92)
-		(end 100.5375 92)
-		(width 0.4)
-		(layer "F.Cu")
-		(net "Net-(C1-Pad1)")
-	)
-	(segment
-		(start 106.4625 91.0375)
-		(end 107.5 90)
-		(width 0.4)
-		(layer "F.Cu")
-		(net "Net-(C1-Pad1)")
-	)
-	(segment
-		(start 104.5 91.0375)
-		(end 106.4625 91.0375)
-		(width 0.4)
-		(layer "F.Cu")
-		(net "Net-(C1-Pad1)")
-	)
-	(segment
-		(start 101.5 91.0375)
-		(end 104.5 91.0375)
-		(width 0.4)
-		(layer "F.Cu")
-		(net "Net-(C1-Pad1)")
-	)
 	(zone

Commit message: V2 보드 완성
Parts:
- removed R3: 0, Resistor_SMD:R_0805_2012Metric_Pad1.20x1.40mm_HandSolder
- added C2: 100uF, Capacitor_Tantalum_SMD:CP_EIA-3528-15_AVX-H_HandSolder, F.Cu at (95.0, 93.5)
- added C4: 100uF, Capacitor_Tantalum_SMD:CP_EIA-3528-15_AVX-H_HandSolder, F.Cu at (108.0, 91.1)
- added FB1: ~, Inductor_SMD:L_0805_2012Metric_Pad1.05x1.20mm_HandSolder, F.Cu at (99.8, 90.0)
- moved C8 13.8 mm to (107.1, 98.8), turned to 90 degrees
- moved C9 13.8 mm to (111.3, 98.8), turned to 90 degrees
- moved C1 9.55 mm to (94.5, 96.5), turned to 0 degrees
- moved C12 8.50 mm to (111.2, 109.8), turned to -90 degrees
- moved C11 8.31 mm to (107.1, 109.5), turned to -90 degrees
- moved R1 7.53 mm to (101.8, 101.8)
- moved R5 7.53 mm to (106.0, 101.8)
- moved R6 7.53 mm to (110.3, 101.8)
- moved R2 2.08 mm to (101.8, 106.7)
- moved R8 2.08 mm to (106.0, 106.7)
- moved R9 2.08 mm to (110.3, 106.7)
- moved R10 1.77 mm to (124.5, 107.0)
- moved R4 1.50 mm to (112.0, 90.0)
- moved C7 1.25 mm to (124.0, 100.0)
- moved C3 1.00 mm to (104.6, 91.0), turned to -90 degrees
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- renumbered C8 to C10, C9 to C11, C10 to C12, C2 to C3, C3 to C5, C4 to C6, C5 to C7, C6 to C8, C7 to C9
Connections:
- C1 pad 1: Net-(C1-Pad1) -> 5V_IN
- C3 pad 1: Net-(C1-Pad1) -> Net-(C3-Pad1)
- R4 pad 2: Net-(C1-Pad1) -> Net-(C3-Pad1)
Routing:
- net Net-(C1-Pad1): track 21.9 -> 0.00 mm
- net 5V_IN: track 3.48 -> 15.2 mm
- net Net-(C3-Pad1): track 0.00 -> 11.6 mm
- net Net-(U2B-+): track 15.5 -> 12.9 mm, vias 2 -> 0
- net GND: track 12.9 -> 11.0 mm, vias 43 -> 53
- net Net-(U2B--): track 7.30 -> 5.51 mm
- net Net-(C10-Pad1): track 6.85 -> 8.26 mm
- net +5V: track 20.8 -> 21.8 mm
- net SDM_R_IN: track 6.12 -> 5.26 mm
- net SDM_L_IN: track 9.58 -> 8.91 mm
