File: pcb/sigma-delta-dac-pcb/sigma-delta-dac-pcb.kicad_pcb (KiCad board)
At the start: 4 copper layers, 60 x 32.5 mm, 50 parts, among them J1 AudioJack3_SwitchTR, J2 Conn_02x03_Top_Bottom, U1 LM27762, U2 SN74LVC1G125DBV, U3 SN74LVC1G125DBV, U4 OPA1688IDR

Commit message: feat: 실크스크린에 로고 & 버전명 추가
Parts:
- added G***: LOGO, Logo:logo, F.Cu at (119.0, 92.0)
Other:
- board text added: "<(Sigma_Delta_v3)"
