File: pcb/sigma-delta-dac-pcb/sim.kicad_sch (KiCad schematic)
At the start: 5 parts, among them U3 ${SIM.PARAMS}

Commit message: v2 회로 - wip
Parts:
- renumbered U3 to U1, V8 to V1, V5 to V2, V7 to V3, V6 to V4
Changed lines of the file:
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@@
 		(in_pos_files yes)
 		(dnp no)
-		(property "Reference" "V5"
+		(property "Reference" "V2"
 			(at 45.72 55.7501 0)
 			(show_name no)
@@
 		(instances
 			(project "sigma-delta-dac-pcb"
-				(path "/b48147e6-cdbe-443e-b50e-c8c9ffc2b6f5"
-					(reference "V5")
+				(path "/a35bdaff-6288-40da-b7db-a5834010c771/d4f48e9e-9982-4ca4-9f98-cecc4545cf7e"
+					(reference "V2")
 					(unit 1)
 				)
@@
 		(in_pos_files yes)
 		(dnp no)
-		(property "Reference" "V7"
+		(property "Reference" "V3"
 			(at 71.12 55.7501 0)
 			(show_name no)
@@
 		(instances
 			(project "sigma-delta-dac-pcb"
-				(path "/b48147e6-cdbe-443e-b50e-c8c9ffc2b6f5"
-					(reference "V7")
+				(path "/a35bdaff-6288-40da-b7db-a5834010c771/d4f48e9e-9982-4ca4-9f98-cecc4545cf7e"
+					(reference "V3")
 					(unit 1)
 				)
@@
 		(in_pos_files yes)
 		(dnp no)
-		(property "Reference" "U3"
+		(property "Reference" "U1"
 			(at 140.97 41.8398 0)
 			(show_name no)
@@
 		(instances
 			(project "sigma-delta-dac-pcb"
-				(path "/b48147e6-cdbe-443e-b50e-c8c9ffc2b6f5"
-					(reference "U3")
+				(path "/a35bdaff-6288-40da-b7db-a5834010c771/d4f48e9e-9982-4ca4-9f98-cecc4545cf7e"
+					(reference "U1")
 					(unit 1)
 				)
@@
 		(dnp no)
 		(fields_autoplaced yes)
-		(property "Reference" "V8"
+		(property "Reference" "V1"
 			(at 170.18 46.8601 0)
 			(show_name no)
@@
 		(instances
 			(project "sigma-delta-dac-pcb"
-				(path "/b48147e6-cdbe-443e-b50e-c8c9ffc2b6f5"
-					(reference "V8")
+				(path "/a35bdaff-6288-40da-b7db-a5834010c771/d4f48e9e-9982-4ca4-9f98-cecc4545cf7e"
+					(reference "V1")
 					(unit 1)
 				)
@@
 		(dnp no)
 		(fields_autoplaced yes)
-		(property "Reference" "V6"
+		(property "Reference" "V4"
 			(at 45.72 102.7401 0)
 			(show_name no)
@@
 		(instances
 			(project "sigma-delta-dac-pcb"
-				(path "/b48147e6-cdbe-443e-b50e-c8c9ffc2b6f5"
-					(reference "V6")
+				(path "/a35bdaff-6288-40da-b7db-a5834010c771/d4f48e9e-9982-4ca4-9f98-cecc4545cf7e"
+					(reference "V4")
 					(unit 1)
 				)
@@
 		(dnp no)
 		(fields_autoplaced yes)
-		(property "Reference" "#PWR015"
+		(property "Reference" "#PWR06"
 			(at 130.81 64.77 0)
 			(hide yes)
@@
 		(instances
 			(project "sigma-delta-dac-pcb"
-				(path "/b48147e6-cdbe-443e-b50e-c8c9ffc2b6f5"
-					(reference "#PWR015")
+				(path "/a35bdaff-6288-40da-b7db-a5834010c771/d4f48e9e-9982-4ca4-9f98-cecc4545cf7e"
+					(reference "#PWR06")
 					(unit 1)
 				)
@@
 		(dnp no)
 		(fields_autoplaced yes)
-		(property "Reference" "#PWR014"
+		(property "Reference" "#PWR08"
 			(at 67.31 73.66 0)
 			(hide yes)
@@
 		(instances
 			(project "sigma-delta-dac-pcb"
-				(path "/b48147e6-cdbe-443e-b50e-c8c9ffc2b6f5"
-					(reference "#PWR014")
+				(path "/a35bdaff-6288-40da-b7db-a5834010c771/d4f48e9e-9982-4ca4-9f98-cecc4545cf7e"
+					(reference "#PWR08")
 					(unit 1)
 				)
@@
 		(dnp no)
 		(fields_autoplaced yes)
-		(property "Reference" "#PWR013"
+		(property "Reference" "#PWR07"
 			(at 41.91 72.39 0)
 			(hide yes)
@@
 		(instances
 			(project "sigma-delta-dac-pcb"
-				(path "/b48147e6-cdbe-443e-b50e-c8c9ffc2b6f5"
-					(reference "#PWR013")
+				(path "/a35bdaff-6288-40da-b7db-a5834010c771/d4f48e9e-9982-4ca4-9f98-cecc4545cf7e"
+					(reference "#PWR07")
 					(unit 1)
 				)
@@
 		)
 	)
-	(sheet_instances
-		(path "/"
-			(page "2")
-		)
-	)

Commit message: V2 보드 완성
Connections:
- net SDM_L renamed SDM_L_IN
Changed lines of the file:
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@@
 		)
 	)
-	(global_label "SDM_L"
+	(global_label "SDM_L_IN"
 		(shape input)
 		(at 148.59 46.99 0)
@@
 		)
 		(property "Intersheetrefs" "${INTERSHEET_REFS}"
-			(at 157.5018 46.99 0)
+			(at 160.4047 46.99 0)
 			(hide yes)
 			(show_name no)
@@
 		(dnp no)
 		(fields_autoplaced yes)
-		(property "Reference" "#PWR06"
+		(property "Reference" "#PWR08"
 			(at 130.81 64.77 0)
 			(hide yes)
@@
 			(project "sigma-delta-dac-pcb"
 				(path "/a35bdaff-6288-40da-b7db-a5834010c771/d4f48e9e-9982-4ca4-9f98-cecc4545cf7e"
-					(reference "#PWR06")
+					(reference "#PWR08")
 					(unit 1)
 				)
@@
 		(dnp no)
 		(fields_autoplaced yes)
-		(property "Reference" "#PWR08"
+		(property "Reference" "#PWR010"
 			(at 67.31 73.66 0)
 			(hide yes)
@@
 			(project "sigma-delta-dac-pcb"
 				(path "/a35bdaff-6288-40da-b7db-a5834010c771/d4f48e9e-9982-4ca4-9f98-cecc4545cf7e"
-					(reference "#PWR08")
+					(reference "#PWR010")
 					(unit 1)
 				)
@@
 		(dnp no)
 		(fields_autoplaced yes)
-		(property "Reference" "#PWR07"
+		(property "Reference" "#PWR09"
 			(at 41.91 72.39 0)
 			(hide yes)
@@
 			(project "sigma-delta-dac-pcb"
 				(path "/a35bdaff-6288-40da-b7db-a5834010c771/d4f48e9e-9982-4ca4-9f98-cecc4545cf7e"
-					(reference "#PWR07")
+					(reference "#PWR09")
 					(unit 1)
 				)
