File: pcb/sigma-delta-dac-pcb/buffer.kicad_sch (KiCad schematic)
At the start: 11 parts, among them U1 LM27762

Commit message: V3 보드 WIP
Parts:
- removed C1, C3: 4.7 uF, Capacitor_SMD:C_0805_2012Metric, symbol Device:C
- removed C2: 1uF, Capacitor_SMD:C_0603_1608Metric, symbol Device:C
- removed C4, C5: 2.2uF, Capacitor_SMD:C_0603_1608Metric, symbol Device:C
- removed D1: ESD9B5.0ST5G, Diode_SMD:D_SOD-923, symbol Diode:ESD9B5.0ST5G
- removed R3: 187 k, Resistor_SMD:R_0603_1608Metric, symbol Device:R_US
- removed R4, R5: 107 k, Resistor_SMD:R_0603_1608Metric, symbol Device:R_US
- removed R6: 182 k, Resistor_SMD:R_0603_1608Metric, symbol Device:R_US
- removed U1: LM27762, Package_SON:WSON-12-1EP_3x2mm_P0.5mm_EP1x2.65_ThermalVias, symbol Regulator_SwitchedCapacitor:LM27762
- added C10: 470 nF, Capacitor_SMD:C_1206_3216Metric, symbol Device:C
- added C11, C8: 2.2nF, Capacitor_SMD:C_0603_1608Metric, symbol Device:C
- added C6, C9: 100nF, Capacitor_SMD:C_0603_1608Metric, symbol Device:C
- added C7: 470nF, Capacitor_SMD:C_1206_3216Metric, symbol Device:C
- added FB1, FB2: FerriteBead, Inductor_SMD:L_0805_2012Metric, symbol Device:FerriteBead
- added R10, R8: 100k, Resistor_SMD:R_0603_1608Metric, symbol Device:R_US
- added R7, R9: 330, Resistor_SMD:R_0603_1608Metric, symbol Device:R_US
- added U2, U3: SN74LVC1G125DBV, Package_TO_SOT_SMD:SOT-23-5, symbol 74xGxx:SN74LVC1G125DBV
Connections:
- net +3V3: now also FB1.1, FB2.1
- net GND: now also C11.2, C6.2, C8.2, C9.2, R10.2, R8.2, U2.1, U2.3 (GND), U3.1, U3.3 (GND)
- new net: C10.1, C11.1, R9.2
- new net: C7.1, C8.1, R7.2
- new net: R9.1, U3.4
- new net: C9.1, FB2.2, U3.5 (VCC)
- new net: C6.1, FB1.2, U2.5 (VCC)
- new net: R7.1, U2.4
- new net BUFFER_L: C7.2, R8.1
- new net BUFFER_R: C10.2, R10.1
- new net SDM_L: U2.2
- new net SDM_R: U3.2

Commit message: 캐패시터 사이즈 변경
Parts:
- C10: value 470 nF -> 470nF
- C6, C9: footprint Capacitor_SMD:C_0603_1608Metric -> Capacitor_SMD:C_0402_1005Metric
Changed lines of the file:
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@@
 			)
 		)
-		(property "Value" "470 nF"
+		(property "Value" "470nF"
 			(at 133.3499 110.49 0)
 			(show_name no)
@@
 			)
 		)
-		(property "Footprint" "Capacitor_SMD:C_0603_1608Metric"
+		(property "Footprint" "Capacitor_SMD:C_0402_1005Metric"
 			(at 63.1952 62.23 0)
 			(hide yes)
@@
 			)
 		)
-		(property "Description" "50V 1608 X7R"
+		(property "Description" "50V 1005 X7R"
 			(at 70.612 61.468 0)
+			(show_name no)
+			(do_not_autoplace no)
+			(effects
+				(font
+					(size 1.27 1.27)
+				)
+			)
+		)
+		(property "Sim.Device" ""
+			(at 62.23 58.42 0)
+			(hide yes)
+			(show_name no)
+			(do_not_autoplace no)
+			(effects
+				(font
+					(size 1.27 1.27)
+				)
+			)
+		)
+		(property "Sim.Library" ""
+			(at 62.23 58.42 0)
+			(hide yes)
+			(show_name no)
+			(do_not_autoplace no)
+			(effects
+				(font
+					(size 1.27 1.27)
+				)
+			)
+		)
+		(property "Sim.Name" ""
+			(at 62.23 58.42 0)
+			(hide yes)
+			(show_name no)
+			(do_not_autoplace no)
+			(effects
+				(font
+					(size 1.27 1.27)
+				)
+			)
+		)
+		(property "Sim.Pins" ""
+			(at 62.23 58.42 0)
+			(hide yes)
 			(show_name no)
 			(do_not_autoplace no)
@@
 			)
 		)
-		(property "Footprint" "Capacitor_SMD:C_0603_1608Metric"
+		(property "Footprint" "Capacitor_SMD:C_0402_1005Metric"
 			(at 63.1952 102.87 0)
 			(hide yes)
@@
 			)
 		)
-		(property "Description" "50V 1608 X7R"
+		(property "Description" "50V 1005 X7R"
 			(at 70.612 102.108 0)
 			(show_name no)
 			(do_not_autoplace no)
+			(effects
+				(font
+					(size 1.27 1.27)
+				)
+			)
+		)
+		(property "Sim.Device" ""
+			(at 62.23 99.06 0)
+			(hide yes)
+			(show_name no)
+			(do_not_autoplace no)
+			(effects
+				(font
+					(size 1.27 1.27)
+				)
+			)
+		)
+		(property "Sim.Library" ""
+			(at 62.23 99.06 0)
+			(hide yes)
+			(show_name no)
+			(do_not_autoplace no)
+			(effects
+				(font
+					(size 1.27 1.27)
+				)
+			)
+		)
+		(property "Sim.Name" ""
+			(at 62.23 99.06 0)
+			(hide yes)
+			(show_name no)
+			(do_not_autoplace no)
+			(effects
+				(font
+					(size 1.27 1.27)
+				)
+			)
+		)
+		(property "Sim.Pins" ""
+			(at 62.23 99.06 0)
+			(hide yes)
+			(show_name no)
+			(do_not_autoplace no)
